File: hardware/pico_adapter/pico_adapter.kicad_sch (KiCad schematic)
At the start: 42 parts, among them J1 L77HDE15SD1CH4F, J2 AudioJack3, J3 5V in, Q1 Q_NMOS_DGS, Q2 Q_NMOS_DGS

Commit message: bigger resistors
Parts:
- R1, R10, R11, R12, R13, R14, R15, R16, R17, R18, R19, R2, R20, R21, R22, R23, R24, R25, R26, R27, R28, R29, R3, R30, R31, R32, R4, R5, R6, R7, R8, R9: footprint Resistor_THT:R_Axial_DIN0204_L3.6mm_D1.6mm_P7.62mm_Horizontal -> Resistor_THT:R_Axial_DIN0207_L6.3mm_D2.5mm_P10.16mm_Horizontal

Commit message: added addon-headers + reset button
Parts:
- removed J3: 5V in, Connector_PinHeader_2.54mm:PinHeader_1x02_P2.54mm_Vertical, symbol Connector:Conn_01x02_Male
- added D1: D_Schottky, Diode_THT:D_A-405_P10.16mm_Horizontal, symbol Device:D_Schottky
- added J4: ADD-ON, Connector_PinHeader_2.54mm:PinHeader_1x09_P2.54mm_Vertical, symbol Connector:Conn_01x09_Male
- added J5: AGND, Connector_PinHeader_2.54mm:PinHeader_1x01_P2.54mm_Vertical, symbol Connector:Conn_01x01_Male
- added J6: PWR_REF, Connector_PinHeader_2.54mm:PinHeader_1x06_P2.54mm_Vertical, symbol Connector:Conn_01x06_Male
- added SW1: SW_Push, Button_Switch_THT:SW_PUSH_6mm_H5mm, symbol Switch:SW_Push
Connections:
- net +3V3: now also J6.2 (Pin_2)
- net +5V: now also D1.2 (A), J6.5 (Pin_5); no longer A1.39 (VSYS)
- net GND: now also J4.1 (Pin_1), J4.6 (Pin_6), J6.4 (Pin_4), SW1.2
- net GPIO17: now reaches A1.22 (GPIO17), R25.2
- net GPIO16: now reaches A1.21 (GPIO16), R26.2
- net GPIO18: now reaches A1.24 (GPIO18)
- net GPIO18: now also J4.2 (Pin_2)
- net GPIO19: now reaches A1.25 (GPIO19)
- net GPIO19: now also J4.3 (Pin_3)
- net GPIO20: now reaches A1.26 (GPIO20)
- net GPIO20: now also J4.4 (Pin_4)
- net GPIO21: now reaches A1.27 (GPIO21)
- net GPIO21: now also J4.5 (Pin_5)
- net GPIO22: now reaches A1.29 (GPIO22)
- net GPIO22: now also J4.7 (Pin_7)
- net RUN: now reaches A1.30 (RUN)
- net RUN: now also J4.8 (Pin_8), SW1.1
- net GPIO26: now reaches A1.31 (GPIO26_ADC0)
- net GPIO26: now also J4.9 (Pin_9)
- net AGND: now reaches A1.33 (AGND)
- net AGND: now also J5.1 (Pin_1)
- net ADC_VREF: now reaches A1.35 (ADC_VREF)
- net ADC_VREF: now also J6.1 (Pin_1)
- net 3V3_EN: now reaches A1.37 (3V3_EN)
- net 3V3_EN: now also J6.3 (Pin_3)
- net VBUS: now reaches A1.40 (VBUS)
- net VBUS: now also J6.6 (Pin_6)
- new net: A1.39 (VSYS), D1.1 (K)
- no-connect marks 16 -> 5
Other:
- note added: "ADD-ON GPIO HEADERS + POWER"
- note added: "Simplified Power Supply circuit: When not using the picos micro USB socket use 5V psu with directly attached wires"
- note added: "TODO: add Low-Pass für Audio Power supply?"
- note added: "VGA_HSYNC"
- note added: "VGA_VSYNC"
- note removed: "POWER"
- note removed: "Simplified Power Supply circuit: Use USB psu with directly attached wires (no micro / type C connectors) OR Use case feed trough with any other basic plugs/sockets"
- moved on the sheet: C1, C2, C4, C5, J1, J2, Q1, Q2, R1, R10, R11, R12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
